File: pcb/Meshbee_receiver.kicad_pro/Meshbee_001.kicad_pro.kicad_pcb (KiCad board)
At the start: 2 copper layers, 42.5 x 100 mm, 14 parts, among them J9 Reset_Button, SW1 button, SW2 reset, U1 Wemos_LoLin32_lite, U2 HT-RA62, U4 nice_nano

Commit message: addedd plot and drill files
Parts:
- removed H5: Hole, MeshBee:MountingHole_5.3mm_M5

Commit message: - transferred some markings on the board to silkscreen layer - renumeration of WEMOS LOLIN32 LITE Pins - modified 3D-printed module for battery - created 3D-print module for MeshBee PCB
Connections:
- U1 pad 14: +3.3V -> /Notifier
- U1 pad 19: unconnected-(U1-5-Pad19) -> /TX
- U1 pad 21: /TX -> unconnected-(U1-5-Pad21)
- U1 pad 26: /Notifier -> +3.3V
Routing:
- net /Notifier: track 14.1 -> 45.6 mm
- net +3.3V: track 103.3 -> 86.3 mm
- net /TX: track 27.8 -> 40.5 mm
- net /RX: track 31.6 -> 33.4 mm
Changed lines of the file:
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@@
 			(unit
 				(name "A")
-				(pins "1" "2" "3" "4" "5" "6" "7" "8" "9" "10" "11" "12" "13" "14" "15"
-					"16" "17" "18" "19" "20" "21" "22" "23" "24" "25" "26"
+				(pins "1" "2" "3" "4" "5" "6" "7" "8" "9" "10" "11" "12" "13" "26" "25"
+					"24" "23" "22" "21" "20" "19" "18" "17" "16" "15" "14"
 				)
 			)
@@
 			(layers "*.Cu" "*.Mask")
 			(remove_unused_layers no)
-			(net "+3.3V")
-			(pinfunction "3V_14")
-			(pintype "power_out")
+			(net "/Notifier")
+			(pinfunction "13_14")
+			(pintype "bidirectional")
 		)
 		(pad "15" thru_hole oval
@@
 			(layers "*.Cu" "*.Mask")
 			(remove_unused_layers no)
-			(net "unconnected-(U1-22-Pad15)")
-			(pinfunction "22_15")
+			(net "unconnected-(U1-Pad15)")
+			(pinfunction "15_15")
 			(pintype "bidirectional+no_connect")
 		)
@@
 			(layers "*.Cu" "*.Mask")
 			(remove_unused_layers no)
-			(net "unconnected-(U1-19-Pad16)")
-			(pinfunction "19_16")
+			(net "unconnected-(U1-2-Pad16)")
+			(pinfunction "2_16")
 			(pintype "bidirectional+no_connect")
 		)
@@
 			(layers "*.Cu" "*.Mask")
 			(remove_unused_layers no)
-			(net "unconnected-(U1-23-Pad17)")
-			(pinfunction "23_17")
+			(net "unconnected-(U1-0-Pad17)")
+			(pinfunction "0_17")
 			(pintype "bidirectional+no_connect")
 		)
@@
 			(layers "*.Cu" "*.Mask")
 			(remove_unused_layers no)
-			(net "unconnected-(U1-Pad18)")
-			(pinfunction "18_18")
+			(net "unconnected-(U1-4-Pad18)")
+			(pinfunction "4_18")
 			(pintype "bidirectional+no_connect")
 		)
@@
 			(layers "*.Cu" "*.Mask")
 			(remove_unused_layers no)
-			(net "unconnected-(U1-5-Pad19)")
-			(pinfunction "5_19")
-			(pintype "bidirectional+no_connect")
+			(net "/TX")
+			(pinfunction "16_19")
+			(pintype "bidirectional")
 		)
 		(pad "20" thru_hole oval
@@
 			(layers "*.Cu" "*.Mask")
 			(remove_unused_layers no)
-			(net "/TX")
-			(pinfunction "16_21")
-			(pintype "bidirectional")
+			(net "unconnected-(U1-5-Pad21)")
+			(pinfunction "5_21")
+			(pintype "bidirectional+no_connect")
 		)
 		(pad "22" thru_hole oval
@@
 			(layers "*.Cu" "*.Mask")
 			(remove_unused_layers no)
-			(net "unconnected-(U1-4-Pad22)")
-			(pinfunction "4_22")
+			(net "unconnected-(U1-18-Pad22)")
+			(pinfunction "18_22")
 			(pintype "bidirectional+no_connect")
 		)
@@
 			(layers "*.Cu" "*.Mask")
 			(remove_unused_layers no)
-			(net "unconnected-(U1-0-Pad23)")
-			(pinfunction "0_23")
+			(net "unconnected-(U1-Pad23)")
+			(pinfunction "23_23")
 			(pintype "bidirectional+no_connect")
 		)
@@
 			(layers "*.Cu" "*.Mask")
 			(remove_unused_layers no)
-			(net "unconnected-(U1-2-Pad24)")
-			(pinfunction "2_24")
+			(net "unconnected-(U1-19-Pad24)")
+			(pinfunction "19_24")
 			(pintype "bidirectional+no_connect")
 		)
@@
 			(layers "*.Cu" "*.Mask")
 			(remove_unused_layers no)
-			(net "unconnected-(U1-15-Pad25)")
-			(pinfunction "15_25")
+			(net "unconnected-(U1-22-Pad25)")
+			(pinfunction "22_25")
 			(pintype "bidirectional+no_connect")
 		)
@@
 			(layers "*.Cu" "*.Mask")
 			(remove_unused_layers no)
-			(net "/Notifier")
-			(pinfunction "13_26")
-			(pintype "bidirectional")
+			(net "+3.3V")
+			(pinfunction "3V_26")
+			(pintype "power_out")
 		)
 		(embedded_fonts no)
@@
 	)
 	(segment
-		(start 86.4 62.634314)
-		(end 86.4 77.7)
+		(start 91.1 60.1)
+		(end 91.1 76.35)
 		(width 0.2)
 		(layer "F.Cu")
@@
 	)
 	(segment
-		(start 82.56 53.595635)
-		(end 83.204365 54.24)
+		(start 82.56 52.96)
+		(end 82.56 53.595635)
+		(width 0.2)
+		(layer "F.Cu")
+		(net "/RX")
+	)
+	(segment
+		(start 90.5 76.95)
+		(end 90.495 76.95)
 		(width 0.2)
 		(layer "F.Cu")
@@
 	(segment
 		(start 83.204365 54.24)
-		(end 83.84 54.24)
+		(end 85.24 54.24)
 		(width 0.2)
 		(layer "F.Cu")
@@
 	)
 	(segment
-		(start 82.34 52.74)
-		(end 82.56 52.96)
+		(start 91.1 76.35)
+		(end 90.5 76.95)
 		(width 0.2)
 		(layer "F.Cu")
@@
 	)
 	(segment
-		(start 87.715 79.015)
-		(end 88.43 79.015)
+		(start 82.56 53.595635)
+		(end 83.204365 54.24)
+		(width 0.2)
+		(layer "F.Cu")
+		(net "/RX")
+	)
+	(segment
+		(start 82.34 52.74)
+		(end 82.56 52.96)
 		(width 0.2)
 		(layer "F.Cu")
@@
 	)
 	(segment
-		(start 82.56 52.96)
-		(end 82.56 53.595635)
+		(start 85.24 54.24)
+		(end 91.1 60.1)
 		(width 0.2)
 		(layer "F.Cu")
@@
 	)
 	(segment
-		(start 87.3 57.7)
-		(end 87.3 61.734314)
+		(start 90.495 76.95)
+		(end 88.43 79.015)
 		(width 0.2)
 		(layer "F.Cu")
@@
 	)
 	(segment
-		(start 83.84 54.24)
-		(end 87.3 57.7)
+		(start 86.65 56.7)
+		(end 86.65 79.775)
 		(width 0.2)
 		(layer "F.Cu")
-		(net "/RX")
+		(net "/TX")
 	)
 	(segment
-		(start 87.3 61.734314)
-		(end 86.4 62.634314)
+		(start 83.66 52.74)
+		(end 81.62 50.7)
 		(width 0.2)
 		(layer "F.Cu")
-		(net "/RX")
+		(net "/TX")
 	)
 	(segment
-		(start 86.4 77.7)
-		(end 87.715 79.015)
+		(start 79.85 53.5)
+		(end 81.3 54.95)
 		(width 0.2)
 		(layer "F.Cu")
-		(net "/RX")
+		(net "/TX")
 	)
 	(segment
-		(start 88.43 76.475)
-		(end 86.8 74.845)
+		(start 80.95 50.7)
+		(end 79.85 51.8)
 		(width 0.2)
 		(layer "F.Cu")
@@
 	)
 	(segment
-		(start 86.8 74.845)
-		(end 86.8 62.8)
+		(start 79.85 51.8)
+		(end 79.85 53.5)
 		(width 0.2)
 		(layer "F.Cu")
@@
 	)
 	(segment
-		(start 86.8 62.8)
-		(end 89.3 60.3)
+		(start 81.3 54.95)
+		(end 84.9 54.95)
 		(width 0.2)
 		(layer "F.Cu")
@@
 	)
 	(segment
-		(start 89.3 58.38)
-		(end 83.66 52.74)
+		(start 84.9 54.95)
+		(end 86.65 56.7)
 		(width 0.2)
 		(layer "F.Cu")
@@
 	)
 	(segment
-		(start 89.3 60.3)
-		(end 89.3 58.38)
+		(start 86.65 79.775)
+		(end 88.43 81.555)
 		(width 0.2)
 		(layer "F.Cu")
@@
 	)
 	(segment
-		(start 88.275 63.775)
-		(end 90.8 61.25)
+		(start 81.62 50.7)
+		(end 80.95 50.7)
 		(width 0.2)
 		(layer "F.Cu")
-		(net "/Notifier")
+		(net "/TX")
 	)
 	(segment
-		(start 90.8 57.34)
-		(end 86.2 52.74)
+		(start 92.3 58.84)
+		(end 92.3 90.385)
 		(width 0.2)
 		(layer "F.Cu")
@@
 	)
 	(segment
-		(start 90.8 61.25)
-		(end 90.8 57.34)
+		(start 92.3 90.385)
+		(end 88.43 94.255)
 		(width 0.2)
 		(layer "F.Cu")
@@
 	)
 	(segment
-		(start 88.43 63.775)
-		(end 88.275 63.775)
+		(start 86.2 52.74)
+		(end 92.3 58.84)
 		(width 0.2)
 		(layer "F.Cu")
@@
 		(net "+3.3V")
 	)
-	(segment
-		(start 88.43 94.255)
-		(end 89.145 94.255)
-		(width 0.2)
-		(layer "F.Cu")
-		(net "+3.3V")
-	)
 	(via
 		(at 75.9 31)
@@
 	)
 	(segment
-		(start 93.7 55.1)
-		(end 78.6 55.1)
+		(start 91.455 60.75)
+		(end 88.43 63.775)
+		(width 0.2)
+		(layer "B.Cu")
+		(net "+3.3V")
+	)
+	(segment
+		(start 99.1 71.9)
+		(end 99.1 61.3)
+		(width 0.2)
+		(layer "B.Cu")
+		(net "+3.3V")
+	)
+	(segment
+		(start 86.7 55.1)
+		(end 88.5 56.9)
 		(width 0.2)
 		(layer "B.Cu")
@@
 	)
 	(segment
-		(start 99.4 60.8)
-		(end 93.7 55.1)
+		(start 98.55 60.75)
+		(end 91.455 60.75)
 		(width 0.2)
 		(layer "B.Cu")
@@
 	)
 	(segment
-		(start 76.4 37.5)
-		(end 76.04 37.5)
+		(start 88.5 56.9)
+		(end 88.43 56.97)
 		(width 0.2)
 		(layer "B.Cu")
@@
 	)
 	(segment
-		(start 99.4 75.5)
-		(end 99.4 60.8)
+		(start 76.4 37.5)
+		(end 76.04 37.5)
 		(width 0.2)
 		(layer "B.Cu")
@@
 	)
 	(segment
-		(start 89.145 94.255)
-		(end 90.5 92.9)
+		(start 88.43 56.97)
+		(end 88.43 63.775)
 		(width 0.2)
 		(layer "B.Cu")
@@
 	)
 	(segment
-		(start 94.5 76.5)
-		(end 98.4 76.5)
+		(start 78.6 55.1)
+		(end 86.7 55.1)
 		(width 0.2)
 		(layer "B.Cu")
@@
 	)
 	(segment
-		(start 90.5 80.5)
-		(end 94.5 76.5)
+		(start 99.1 61.3)
+		(end 98.55 60.75)
 		(width 0.2)
 		(layer "B.Cu")
@@
 	)
 	(segment
-		(start 90.5 92.9)
-		(end 90.5 80.5)
+		(start 94.5 76.5)
+		(end 99.1 71.9)
 		(width 0.2)
 		(layer "B.Cu")
@@
 		(width 0.2)
 		(layer "B.Cu")
-		(net "+3.3V")
-	)
-	(segment
-		(start 98.4 76.5)
-		(end 99.4 75.5)
-		(width 0.2)
-		(layer "B.Cu")
