File: pcb/Meshbee_receiver.kicad_pro/Meshbee_001.kicad_pro.kicad_sch (KiCad schematic)
At the start: 11 parts, among them J9 Reset_Button, SW1 button, SW2 reset, U1 Wemos_LoLin32_lite, U2 HT-RA62, U4 nice_nano

Commit message: - transferred some markings on the board to silkscreen layer - renumeration of WEMOS LOLIN32 LITE Pins - modified 3D-printed module for battery - created 3D-print module for MeshBee PCB
Connections:
- net +3.3V: now also U1.26 (3V); no longer U1.14 (3V)
- net Notifier: now also U1.14 (13); no longer U1.26 (13)
- net TX: now also U1.19 (16); no longer U1.21 (16)
